File: hardware/kicad/ContainerLevelSensor/ContainerLevelSensor.kicad_pcb (KiCad board)
At the start: 2 copper layers, 44 x 80 mm, 8 parts, among them U1 HW-373, U2 ESP32-C3-SuperMini, U3 VL53LDK, U4 S09

Commit message: Added version 1.1
Parts:
- moved U4 1.58 mm to (180.6, 71.6)
Routing:
- net Net-(U1-OUT+): track 6.83 -> 8.41 mm
- net Net-(JP2-B): track 52.3 -> 53.2 mm
Other:
- board text added: "Container"
- board text added: "Level"
- board text added: "Sensor"
